File: curcuit/esp32_mpboard.sch (EAGLE design)
At the start: 13 parts, among them IC1 TPS6300, IC2 NJM12888F1812DBV, U1 ESP32-WROVER-B_(16MB), U2 CODECODER-VS1053B(LQFP48)

Commit message: ・SDカード読み込み処理を追加 ・ガーバーファイルを更新
Parts:
- added C10, C9: (no value), rcl:C-USC0603
- added C11, C13: 10nF, rcl:C-USC0603
- added C12: 47nF, rcl:C-USC0603
- added C14, C30, C32, C33, C7: 1uF, rcl:C-USC0603
- added C15, C19, C23, C29, C31, C8: 10uF, rcl:C-USC0805
- added C16, C17, C18, C20, C21, C22, C24, C25, C26, C27, C28: 0.1uF, rcl:C-USC0603
- added C6: 0.47uF, rcl:C-USC0603
- added CN1: (no value), jst-xh:B3B-XH-A
- added CN2: (no value), jst-xh:B2B-XH-A
- added J1: PJ-3420-A-SMT, PJ-3420-A-SMT:PJ-3420-A-SMT
- added J2: MEM2075-00-140-01-A, MEM2075-00-140-01-A:MEM2075-00-140-01-A
- added R10: 100k, rcl:R-US_R0603
- added R11, R12: 10k, rcl:R-US_R0603
- added R13, R16, R17, R4, R5: (no value), rcl:R-US_R0603
- added R14, R15: 470R, rcl:R-US_R0603
- added R18, R19, R20: 100Ω, rcl:R-US_R0603
- added R6: 1M, rcl:R-US_R0603
- added R7, R9: 20R, rcl:R-US_R0603
- added R8: 10R, rcl:R-US_R0603
- added S1, S2: MOMENTARY-SWITCH-SPST-SMD-5.2-REDUNDANT, SparkFun-Switches:MOMENTARY-SWITCH-SPST-SMD-5.2-REDUNDANT
- added S3: (no value), SparkFun-Switches:SWITCH-SPDT-PTH-11.6X4.0MM
- added X1: CRYSTALS-NOGND-HC49, IQD-Frequency-Products:CRYSTALS-NOGND-HC49
- C1, C5: value (none) -> 0.1uF
- C2, C3, C4: value (none) -> 10uF
- IC1: value TPS6300 -> TPS63000; device texas:TPS6300 -> TPS63000:TPS63000
- R1: value (none) -> 100Ω
- U1: value ESP32-WROVER-B_(16MB) -> ESP-WROOM-32; device ESP32-WROVER-B__16MB_:ESP32-WROVER-B_(16MB) -> esp32:ESP-WROOM-32
Connections:
- new net 1.8V1: C9.1, R6.2, U2.XTALO, X1.2
- new net 3V3: C15.1, C16.1, C17.1, C18.1, C19.1, C2.1, C20.1, C21.1, C22.1, C27.1, C29.1, C3.1, C30.1, C31.1, C32.1, C5.1, C8.1, IC1G$1.VOUT, IC2.CONTROL, IC2.IN, J2.VDD, R12.2, R18.2, R19.2, R3.2, R5.1, R5.2, U1.3V3, U2.AVDD0, U2.AVDD1, U2.AVDD2, U2.IOVDD0, U2.IOVDD1, U2.IOVDD2, U2.RX
- new net AUDIO_RESET: R10.2, U1.IO5, U2.XRESET
- new net GND1: C10.1, R6.1, U2.XTALI, X1.1
- new net N$12: C12.1, R8.2
- new net N$13: C13.1, R9.2
- new net N$14: C11.1, R7.2
- new net N$15: R12.1, R15.2, U1.IO0
- new net N$16: C14.1, U2.RCAP
- new net N$17: C28.1, R11.1, R14.2, S2.2
- new net N$18: R13.2, U1.IO2
- new net N$20: R14.1, U1.EN
- new net N$21: R15.1, S1.1
- new net N$6: J1.4, R9.1, U2.LEFT
- new net N$8: J1.1, J1.2, R8.1, U2.GBUF
- new net N$9: J1.3, R7.1, U2.RIGHT
- new net SD_CS: J2.CD/DAT3, U1.IO26
- new net SD_MISO: J2.DAT0, R19.1, U1.IO27
- new net SD_MOSI: J2.CMD, R18.1, U1.IO13
- new net SD_SCLK: J2.CLK, R20.2, U1.IO14
- new net UART_RX: CN1.2, U1.RXD0
- new net UART_TX: CN1.1, U1.TXD0
- new net VDD_AD: C33.1, R16.1, R17.2, U1.IO33
- new net VS1053B_DREQ: U1.IO17, U2.DREQ
- new net VS1053B_GPIO: R4.2, U2.GPIO0, U2.GPIO1, U2.GPIO2/DCLK1, U2.GPIO3/SDATA1, U2.GPIO4/I2S-LROUT3, U2.GPIO6/I2S_SCLK3, U2.GPIO7/I2S_SDATA3
- new net VS1053B_MISO: U1.IO19, U2.SO
- new net VS1053B_MOSI: U1.IO23, U2.SI
- new net VS1053B_SCLK: U1.IO18, U2.SCLK
- new net VS1053B_XCS: U1.IO4, U2.XCS
- new net VS1053B_XDCS: U1.IO16, U2.XDCS/BSYNC1
- new net V_BATT: CN2.1, S3.O, S3.P
- net +3V3: now also R11.2; no longer C2.1, C3.1, C5.1, IC1G$1.VOUT, IC2.CONTROL, IC2.IN, R3.2
- net 1.8V: now also C23.1, C24.1, C25.1, C26.1, C6.1, C7.1, U2.CVDD0, U2.CVDD1, U2.CVDD2, U2.CVDD3
- net GND: now also C10.2, C11.2, C12.2, C13.2, C14.2, C15.2, C16.2, C17.2, C18.2, C19.2, C20.2, C21.2, C22.2, C23.2, C24.2, C25.2, C26.2, C27.2, C28.2, C29.2, C30.2, C31.2, C32.2, C33.2, C6.2, C7.2, C8.2, C9.2, CN1.3, CN2.2, J2.VSS, R10.1, R13.1, R17.1, R20.1, R4.1, S1.2, S2.1, U1.GND@1, U1.GND@15, U1.GND@38, U2.AGND0, U2.AGND1, U2.AGND2, U2.AGND3, U2.DGND0, U2.DGND1, U2.DGND2, U2.DGND3, U2.DGND4, U2.GND
- net VDD: now also R16.2, S3.S
Other:
- moved on the sheet: U2
